File: Episode 1 - The 6309 basics and more/CPU.kicad_sch (KiCad schematic)
At the start: 22 parts, among them U1 74AHCT541, U2 74AHCT245, U3 HD63C09, U4 74AHCT541, U5 74AHCT541, U6 ATF750C, Y1 14.31818 MHz, Y2 20 MHz

Commit message: Dropped the curved traces
Parts:
- added SW1: RESET, Button_Switch_THT:SW_Tactile_SPST_Angled_PTS645Vx39-2LFS, symbol Switch:SW_Push
Connections:
- net GND: now also SW1.2
- net ~{RESET}: now also SW1.1
Changed lines of the file:
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@@
 	)
 	(junction
+		(at 57.15 31.75)
+		(diameter 0)
+		(color 0 0 0 0)
+	)
+	(junction
 		(at 54.61 68.58)
 		(diameter 0)
@@
 		)
 	)
+	(wire
+		(pts
+			(xy 57.15 31.75) (xy 60.96 31.75)
+		)
+		(stroke
+			(width 0)
+			(type default)
+		)
+	)
 	(bus
 		(pts
@@
 	(wire
 		(pts
+			(xy 57.15 44.45) (xy 57.15 45.72)
+		)
+		(stroke
+			(width 0)
+			(type default)
+		)
+	)
+	(wire
+		(pts
 			(xy 130.81 43.18) (xy 124.46 43.18)
 		)
@@
 	(wire
 		(pts
+			(xy 57.15 31.75) (xy 57.15 34.29)
+		)
+		(stroke
+			(width 0)
+			(type default)
+		)
+	)
+	(wire
+		(pts
 			(xy 60.96 123.19) (xy 109.22 123.19)
 		)
@@
 	(wire
 		(pts
-			(xy 49.53 31.75) (xy 60.96 31.75)
+			(xy 49.53 31.75) (xy 57.15 31.75)
 		)
 		(stroke
@@
 		(on_board yes)
 		(dnp no)
-		(property "Reference" "#PWR013"
+		(property "Reference" "#PWR014"
 			(at 41.91 132.08 0)
 			(effects
@@
 			(project "Episode 1 - The 6309 basics and more"
 				(path "/5aeeb5e8-9d85-437a-bcb8-c2a3d321d580/09cbd9d8-b4d6-483c-bf1a-da195c518008"
-					(reference "#PWR013")
+					(reference "#PWR014")
 					(unit 1)
 				)
@@
 		(on_board yes)
 		(dnp no)
-		(property "Reference" "#PWR06"
+		(property "Reference" "#PWR07"
 			(at 46.99 57.15 0)
 			(effects
@@
 			(project "Episode 1 - The 6309 basics and more"
 				(path "/5aeeb5e8-9d85-437a-bcb8-c2a3d321d580/09cbd9d8-b4d6-483c-bf1a-da195c518008"
-					(reference "#PWR06")
+					(reference "#PWR07")
 					(unit 1)
 				)
@@
 		(on_board yes)
 		(dnp no)
-		(property "Reference" "#PWR024"
+		(property "Reference" "#PWR025"
 			(at 125.73 198.12 0)
 			(effects
@@
 			(project "Episode 1 - The 6309 basics and more"
 				(path "/5aeeb5e8-9d85-437a-bcb8-c2a3d321d580/09cbd9d8-b4d6-483c-bf1a-da195c518008"
-					(reference "#PWR024")
+					(reference "#PWR025")
 					(unit 1)
 				)
@@
 		(on_board yes)
 		(dnp no)
-		(property "Reference" "#PWR023"
+		(property "Reference" "#PWR024"
 			(at 125.73 185.42 0)
 			(effects
@@
 			(project "Episode 1 - The 6309 basics and more"
 				(path "/5aeeb5e8-9d85-437a-bcb8-c2a3d321d580/09cbd9d8-b4d6-483c-bf1a-da195c518008"
-					(reference "#PWR023")
+					(reference "#PWR024")
 					(unit 1)
 				)
@@
 		(on_board yes)
 		(dnp no)
-		(property "Reference" "#PWR011"
+		(property "Reference" "#PWR012"
 			(at 212.09 110.49 0)
 			(effects
@@
 			(project "Episode 1 - The 6309 basics and more"
 				(path "/5aeeb5e8-9d85-437a-bcb8-c2a3d321d580/09cbd9d8-b4d6-483c-bf1a-da195c518008"
-					(reference "#PWR011")
+					(reference "#PWR012")
 					(unit 1)
 				)
@@
 		(on_board yes)
 		(dnp no)
-		(property "Reference" "#PWR012"
+		(property "Reference" "#PWR013"
 			(at 88.9 116.84 0)
 			(effects
@@
 			(project "Episode 1 - The 6309 basics and more"
 				(path "/5aeeb5e8-9d85-437a-bcb8-c2a3d321d580/09cbd9d8-b4d6-483c-bf1a-da195c518008"
-					(reference "#PWR012")
+					(reference "#PWR013")
 					(unit 1)
 				)
@@
 		(on_board yes)
 		(dnp no)
-		(property "Reference" "#PWR021"
+		(property "Reference" "#PWR022"
 			(at 29.21 186.69 0)
 			(effects
@@
 			(project "Episode 1 - The 6309 basics and more"
 				(path "/5aeeb5e8-9d85-437a-bcb8-c2a3d321d580/09cbd9d8-b4d6-483c-bf1a-da195c518008"
-					(reference "#PWR021")
+					(reference "#PWR022")
 					(unit 1)
 				)
@@
 		(on_board yes)
 		(dnp no)
-		(property "Reference" "#PWR019"
+		(property "Reference" "#PWR020"
 			(at 41.91 163.83 0)
 			(effects
@@
 			(project "Episode 1 - The 6309 basics and more"
 				(path "/5aeeb5e8-9d85-437a-bcb8-c2a3d321d580/09cbd9d8-b4d6-483c-bf1a-da195c518008"
-					(reference "#PWR019")
+					(reference "#PWR020")
 					(unit 1)
 				)
@@
 		(on_board yes)
 		(dnp no)
-		(property "Reference" "#PWR015"
+		(property "Reference" "#PWR016"
 			(at 88.9 142.24 0)
 			(effects
@@
 			(project "Episode 1 - The 6309 basics and more"
 				(path "/5aeeb5e8-9d85-437a-bcb8-c2a3d321d580/09cbd9d8-b4d6-483c-bf1a-da195c518008"
-					(reference "#PWR015")
+					(reference "#PWR016")
 					(unit 1)
 				)
@@
 		(on_board yes)
 		(dnp no)
-		(property "Reference" "#PWR018"
+		(property "Reference" "#PWR019"
 			(at 212.09 153.67 0)
 			(effects
@@
 			(project "Episode 1 - The 6309 basics and more"
 				(path "/5aeeb5e8-9d85-437a-bcb8-c2a3d321d580/09cbd9d8-b4d6-483c-bf1a-da195c518008"
-					(reference "#PWR018")
+					(reference "#PWR019")
 					(unit 1)
 				)
@@
 		(on_board yes)
 		(dnp no)
-		(property "Reference" "#PWR020"
+		(property "Reference" "#PWR021"
 			(at 29.21 173.99 0)
 			(effects
@@
 			(project "Episode 1 - The 6309 basics and more"
 				(path "/5aeeb5e8-9d85-437a-bcb8-c2a3d321d580/09cbd9d8-b4d6-483c-bf1a-da195c518008"
-					(reference "#PWR020")
+					(reference "#PWR021")
 					(unit 1)
 				)
@@
 		(on_board yes)
 		(dnp no)
-		(property "Reference" "#PWR07"
+		(property "Reference" "#PWR08"
 			(at 143.51 82.55 0)
 			(effects
@@
 			(project "Episode 1 - The 6309 basics and more"
 				(path "/5aeeb5e8-9d85-437a-bcb8-c2a3d321d580/09cbd9d8-b4d6-483c-bf1a-da195c518008"
-					(reference "#PWR07")
+					(reference "#PWR08")
 					(unit 1)
 				)
@@
 		(on_board yes)
 		(dnp no)
-		(property "Reference" "#PWR022"
+		(property "Reference" "#PWR023"
 			(at 88.9 187.96 0)
 			(effects
@@
 			(project "Episode 1 - The 6309 basics and more"
 				(path "/5aeeb5e8-9d85-437a-bcb8-c2a3d321d580/09cbd9d8-b4d6-483c-bf1a-da195c518008"
-					(reference "#PWR022")
+					(reference "#PWR023")
 					(unit 1)
 				)
@@
 	)
 	(symbol
+		(lib_id "power:GND")
+		(at 57.15 45.72 0)
+		(unit 1)
+		(exclude_from_sim no)
+		(in_bom yes)
+		(on_board yes)
+		(dnp no)
+		(property "Reference" "#PWR06"
+			(at 57.15 52.07 0)
+			(effects
+				(font
+					(size 1.27 1.27)
+				)
+				(hide yes)
+			)
+		)
+		(property "Value" "GND"
+			(at 57.15 49.53 0)
+			(effects
+				(font
+					(size 1.27 1.27)
+				)
+			)
+		)
+		(property "Footprint" ""
+			(at 57.15 45.72 0)
+			(effects
+				(font
+					(size 1.27 1.27)
+				)
+				(hide yes)
+			)
+		)
+		(property "Datasheet" ""
+			(at 57.15 45.72 0)
+			(effects
+				(font
+					(size 1.27 1.27)
+				)
+				(hide yes)
+			)
+		)
+		(property "Description" "Power symbol creates a global label with name \"GND\" , ground"
+			(at 57.15 45.72 0)
+			(effects
+				(font
+					(size 1.27 1.27)
+				)
+				(hide yes)
+			)
+		)
+		(pin "1"
+		)
+		(instances
+			(project "Episode 1 - The 6309 basics and more"
+				(path "/5aeeb5e8-9d85-437a-bcb8-c2a3d321d580/09cbd9d8-b4d6-483c-bf1a-da195c518008"
+					(reference "#PWR06")
+					(unit 1)
+				)
+			)
+		)
+	)
+	(symbol
 		(lib_id "Device:C_Small")
 		(at 46.99 175.26 0)
@@
 		(on_board yes)
 		(dnp no)
-		(property "Reference" "#PWR016"
+		(property "Reference" "#PWR017"
 			(at 190.5 147.32 0)
 			(effects
@@
 			(project "Episode 1 - The 6309 basics and more"
 				(path "/5aeeb5e8-9d85-437a-bcb8-c2a3d321d580/09cbd9d8-b4d6-483c-bf1a-da195c518008"
-					(reference "#PWR016")
+					(reference "#PWR017")
 					(unit 1)
 				)
@@
 		(on_board yes)
 		(dnp no)
-		(property "Reference" "#PWR08"
+		(property "Reference" "#PWR09"
 			(at 212.09 82.55 0)
 			(effects
@@
 			(project "Episode 1 - The 6309 basics and more"
 				(path "/5aeeb5e8-9d85-437a-bcb8-c2a3d321d580/09cbd9d8-b4d6-483c-bf1a-da195c518008"
-					(reference "#PWR08")
+					(reference "#PWR09")
 					(unit 1)
 				)
@@
 		(on_board yes)
 		(dnp no)
-		(property "Reference" "#PWR014"
+		(property "Reference" "#PWR015"
 			(at 41.91 142.24 0)
 			(effects
@@
 			(project "Episode 1 - The 6309 basics and more"
 				(path "/5aeeb5e8-9d85-437a-bcb8-c2a3d321d580/09cbd9d8-b4d6-483c-bf1a-da195c518008"
-					(reference "#PWR014")
+					(reference "#PWR015")
 					(unit 1)
 				)
@@
 	)
 	(symbol
+		(lib_id "Switch:SW_Push")
+		(at 57.15 39.37 90)
+		(mirror x)
+		(unit 1)
+		(exclude_from_sim no)
+		(in_bom yes)
+		(on_board yes)
+		(dnp no)
+		(property "Reference" "SW1"
+			(at 54.864 38.1 90)
+			(effects
+				(font
+					(size 1.27 1.27)
+				)
+				(justify left)
+			)
+		)
+		(property "Value" "RESET"
+			(at 54.864 40.894 90)
+			(effects
+				(font
+					(size 1.27 1.27)
+				)
+				(justify left)
+			)
+		)
+		(property "Footprint" "Button_Switch_THT:SW_Tactile_SPST_Angled_PTS645Vx39-2LFS"
+			(at 52.07 39.37 0)
+			(effects
+				(font
+					(size 1.27 1.27)
+				)
+				(hide yes)
+			)
+		)
+		(property "Datasheet" "~"
+			(at 52.07 39.37 0)
+			(effects
+				(font
+					(size 1.27 1.27)
+				)
+				(hide yes)
+			)
+		)
+		(property "Description" "Push button switch, generic, two pins"
+			(at 57.15 39.37 0)
+			(effects
+				(font
+					(size 1.27 1.27)
+				)
+				(hide yes)
+			)
+		)
+		(pin "1"
+		)
+		(pin "2"
+		)
+		(instances
+			(project ""
+				(path "/5aeeb5e8-9d85-437a-bcb8-c2a3d321d580/09cbd9d8-b4d6-483c-bf1a-da195c518008"
+					(reference "SW1")
+					(unit 1)
+				)
+			)
+		)
+	)
+	(symbol
 		(lib_id "Oscillator:CXO_DIP8")
 		(at 41.91 116.84 0)
@@
 		(on_board yes)
 		(dnp no)
-		(property "Reference" "#PWR010"
+		(property "Reference" "#PWR011"
 			(at 143.51 110.49 0)
 			(effects
@@
 			(project "Episode 1 - The 6309 basics and more"
 				(path "/5aeeb5e8-9d85-437a-bcb8-c2a3d321d580/09cbd9d8-b4d6-483c-bf1a-da195c518008"
-					(reference "#PWR010")
+					(reference "#PWR011")
 					(unit 1)
 				)
@@
 		(on_board yes)
 		(dnp no)
-		(property "Reference" "#PWR017"
+		(property "Reference" "#PWR018"
 			(at 143.51 153.67 0)
 			(effects
@@
 			(project "Episode 1 - The 6309 basics and more"
 				(path "/5aeeb5e8-9d85-437a-bcb8-c2a3d321d580/09cbd9d8-b4d6-483c-bf1a-da195c518008"
-					(reference "#PWR017")
+					(reference "#PWR018")
 					(unit 1)
 				)
@@
 		(on_board yes)
 		(dnp no)
-		(property "Reference" "#PWR09"
+		(property "Reference" "#PWR010"
 			(at 41.91 110.49 0)
 			(effects
@@
 			(project "Episode 1 - The 6309 basics and more"
 				(path "/5aeeb5e8-9d85-437a-bcb8-c2a3d321d580/09cbd9d8-b4d6-483c-bf1a-da195c518008"
-					(reference "#PWR09")
+					(reference "#PWR010")
 					(unit 1)
 				)

Commit message: PLD coding
Parts:
- added LED1: SPEED, PCM_LED_THT_AKL:LED_D5.0mm-4_RGB_Wide_Pins, symbol PCM_LED_AKL:LED_5mm_RGB_Kcom_RKGB
- added R1: 150, Resistor_THT:R_Axial_DIN0204_L3.6mm_D1.6mm_P5.08mm_Horizontal, symbol Device:R_Small_US
- added R2: 270, Resistor_THT:R_Axial_DIN0204_L3.6mm_D1.6mm_P5.08mm_Horizontal, symbol Device:R_Small_US
- added R3: 330, Resistor_THT:R_Axial_DIN0204_L3.6mm_D1.6mm_P5.08mm_Horizontal, symbol Device:R_Small_US
Connections:
- net SPD_{LED}^{B} is gone; now on net BA5: U6.15 (I/O)
- net SPD_{LED}^{G} is gone; now on net BA4: U6.16 (I/O)
- net SPD_{LED}^{R} is gone; now on net BA3: U6.17 (I/O)
- net BA3: now also R1.1
- net BA4: now also R2.1
- net BA5: now also R3.1
- net GND: now also LED1.2 (A)
- new net: LED1.1 (R), R1.2
- new net: LED1.3 (G), R2.2
- new net: LED1.4 (B), R3.2
Other:
- moved on the sheet: C5, C6, C7, C8
